File: HUB75Adapter.kicad_pcb (KiCad board)
At the start: 2 copper layers, 100 x 100 mm, 14 parts, among them J1 Panel 1, J2 Panel 2, J3 P0_SELECT_PIN4, J4 P0_SELECT_PIN8, J5 P1_SELECT_PIN4, J6 P1_SELECT_PIN8, U1 RaspberryPi Zero WH, U2 74HCT245, U3 74HCT245, U4 74HCT245

Commit message: Initial commit
Parts:
- added C1: 10uF 16V, Capacitor_SMD:C_1206_3216Metric_Pad1.33x1.80mm_HandSolder, F.Cu at (60.7, 123.2)
- added C2: 100nF 50V, Capacitor_SMD:C_1206_3216Metric_Pad1.33x1.80mm_HandSolder, F.Cu at (60.7, 126.5)
- U1: value RaspberryPi Zero WH -> RaspberryPi Zero W
- renumbered C1 to C3, C2 to C4, C3 to C5

Commit message: Add README. Board updates.
Parts:
- added C1: 100nF 50V, Capacitor_SMD:C_1206_3216Metric_Pad1.33x1.80mm_HandSolder, F.Cu at (74.4, 41.9)
- added C10: 1200uF 16V, Capacitor_THT:CP_Radial_D10.0mm_P5.00mm, F.Cu at (141.0, 128.6)
- added C11: 1200uF 16V, Capacitor_THT:CP_Radial_D10.0mm_P5.00mm, F.Cu at (59.0, 128.5)
- added C2: 100nF 50V, Capacitor_SMD:C_1206_3216Metric_Pad1.33x1.80mm_HandSolder, F.Cu at (74.4, 45.2)
- added C4: 1200uF 16V, Capacitor_THT:CP_Radial_D10.0mm_P5.00mm, F.Cu at (141.9, 73.0)
- added C5: 1200uF 16V, Capacitor_THT:CP_Radial_D10.0mm_P5.00mm, F.Cu at (141.9, 62.0)
- added F1: Fuse, Fuse:Fuseholder_Littelfuse_Nano2_154x, F.Cu at (81.0, 138.2)
- added J1: Power input, TerminalBlock_Phoenix:TerminalBlock_Phoenix_MKDS-1,5-4_1x04_P5.00mm_Horizontal, F.Cu at (92.0, 138.3)
- added J2: I2C Extension, Connector_IDC:IDC-Header_2x03_P2.54mm_Vertical, F.Cu at (56.5, 80.3)
- added J5: Screw_Terminal_01x04, TerminalBlock_Phoenix:TerminalBlock_Phoenix_MKDS-1,5-4_1x04_P5.00mm_Horizontal, F.Cu at (145.3, 122.5)
- added J6: Screw_Terminal_01x04, TerminalBlock_Phoenix:TerminalBlock_Phoenix_MKDS-1,5-4_1x04_P5.00mm_Horizontal, F.Cu at (54.7, 107.5)
- added LED1: LED DUAL, PCM_LED_THT_AKL:LED_D3.0mm_BiDir, F.Cu at (55.2, 63.0)
- added Q1: AOD403, PCM_Package_TO_SOT_SMD_AKL:TO-252-2, F.Cu at (70.5, 136.2)
- added R1: 150R, PCM_Resistor_SMD_AKL:R_1206_3216Metric_Pad1.42x1.75mm_HandSolder, F.Cu at (61.2, 64.2)
- added R3: 10k, PCM_Resistor_SMD_AKL:R_1206_3216Metric_Pad1.42x1.75mm_HandSolder, F.Cu at (91.8, 85.8)
- moved C3 73.3 mm to (120.8, 84.5)
- moved C6 38.4 mm to (81.8, 91.0), turned to 90 degrees
- moved C9 8.53 mm to (142.5, 86.8), turned to 180 degrees
- moved J7 4.37 mm to (117.2, 120.5)
- moved J8 4.37 mm to (112.0, 120.5)
- moved J4 4.00 mm to (93.9, 111.2)
- moved C7 3.00 mm to (81.8, 97.0)
- moved J10 1.25 mm to (81.5, 120.5)
- moved J9 1.25 mm to (86.8, 120.5)
- renumbered C2 to C3, C1 to C6, C3 to C7, C4 to C8, C5 to C9, J6 to J10, J1 to J3, J2 to J4, J3 to J7, J4 to J8, J5 to J9, R1 to R2
Connections:
- C3 pad 1: unconnected-(C2-Pad1) -> GND
- C3 pad 2: unconnected-(C2-Pad2) -> +5V
- C6 pad 1: unconnected-(C1-Pad1) -> +5V
- C6 pad 2: unconnected-(C1-Pad2) -> GND
- R2 pad 1: +3.3V -> Net-(U1-3V3_1)
- U1 pad 1: +3.3V -> Net-(U1-3V3_1)
- U1 pad 3: unconnected-(U1-GPIO2/SDA1-Pad3) -> SDA
- U1 pad 36: unconnected-(U1-GPIO16-Pad36) -> LED2
- U1 pad 37: unconnected-(U1-GPIO26-Pad37) -> LED1
- U1 pad 5: unconnected-(U1-GPIO3/SCL-Pad5) -> SCL
- U3 pad 13: unconnected-(U3-B5-Pad13) -> BUF_ROW_E
- U3 pad 14: unconnected-(U3-B4-Pad14) -> BUF_ROW_D
- U3 pad 15: unconnected-(U3-B3-Pad15) -> BUF_ROW_C
- U3 pad 16: unconnected-(U3-B2-Pad16) -> BUF_ROW_B
- U3 pad 17: unconnected-(U3-B1-Pad17) -> BUF_ROW_A
- U3 pad 6: unconnected-(U3-A4-Pad6) -> ROW_D
- U3 pad 7: unconnected-(U3-A5-Pad7) -> ROW_E
- U3 pad 8: ROW_D -> Net-(U3-A6)
- U4 pad 13: unconnected-(U4-B5-Pad13) -> BUF_P0_B2
- U4 pad 14: unconnected-(U4-B4-Pad14) -> BUF_P0_R2
- U4 pad 15: unconnected-(U4-B3-Pad15) -> BUF_P0_G2
- U4 pad 16: unconnected-(U4-B2-Pad16) -> BUF_P0_B1
- U4 pad 17: unconnected-(U4-B1-Pad17) -> BUF_P0_R1
- U4 pad 18: unconnected-(U4-B0-Pad18) -> BUF_P0_G1
- U4 pad 2: unconnected-(U4-A0-Pad2) -> P0_G1
- U4 pad 3: unconnected-(U4-A1-Pad3) -> P0_R1
- U4 pad 4: unconnected-(U4-A2-Pad4) -> P0_B1
- U4 pad 5: unconnected-(U4-A3-Pad5) -> P0_G2
- U4 pad 6: unconnected-(U4-A4-Pad6) -> P0_R2
- U4 pad 7: unconnected-(U4-A5-Pad7) -> P0_B2
Routing:
- net +5V: track 115.4 -> 278.2 mm, vias 1 -> 5
- net SCL: track 0.00 -> 82.0 mm, vias 0 -> 1
- net SDA: track 0.00 -> 81.5 mm, vias 0 -> 1
- net P0_B1: track 2.81 -> 73.2 mm
- net +3.3V: track 5.59 -> 75.4 mm, vias 0 -> 1
- net P0_R2: track 1.77 -> 65.9 mm
- net P0_R1: track 4.78 -> 59.8 mm
- net P0_G2: track 5.71 -> 52.5 mm
- net P0_B2: track 4.94 -> 49.0 mm
- net P0_G1: track 1.81 -> 45.1 mm, vias 0 -> 2
- net Net-(U1-3V3_1): track 0.00 -> 29.7 mm
- net ROW_E: track 0.00 -> 25.5 mm, vias 0 -> 1
- net BUF_ROW_E: track 39.2 -> 64.2 mm, vias 0 -> 2
- net BUF_P0_G1: track 0.00 -> 22.6 mm
- net BUF_ROW_D: track 40.8 -> 61.8 mm, vias 1 -> 3
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- added copper zone on B.Cu, net +5V
- added copper zone on F.Cu, net +5V
- added copper zone on F.Cu, net Net-(J1-Pin_1)
- added copper zone on F.Cu, net Net-(Q1-D)
Other:
- board size 100 x 100 mm -> 100 x 93 mm
- board text added: "+5V"
- board text added: "I2C Extension"
- board text added: "INPUT PWR"
- board text added: "PANEL PWR"

Commit message: Finish board
Parts:
- added G***: LOGO, LOGO, F.Cu at (100.0, 103.5)
- added G***: LOGO, LOGO, B.Cu at (87.5, 66.0)
- added G***: LOGO, LOGO, B.Cu at (111.0, 65.5)
- added G***: LOGO, LOGO, B.Cu at (98.5, 65.0)
- added J1: Power input, Connector_BarrelJack:BarrelJack_Horizontal, F.Cu at (126.2, 129.2)
- added R1: 3k3, PCM_Resistor_SMD_AKL:R_1206_3216Metric_Pad1.42x1.75mm_HandSolder, F.Cu at (132.2, 62.8)
- added R2: 3k3, PCM_Resistor_SMD_AKL:R_1206_3216Metric_Pad1.42x1.75mm_HandSolder, F.Cu at (132.2, 68.8)
- added TP1: TP+5V, TestPoint:TestPoint_Pad_D1.0mm, F.Cu at (145.5, 82.0)
- added TP2: TPGND, TestPoint:TestPoint_Pad_D1.0mm, F.Cu at (145.5, 78.8)
- added TP3: TP+3.3V, TestPoint:TestPoint_Pad_D1.0mm, F.Cu at (127.0, 85.0)
- C1, C6, C7, C8, C9: footprint Capacitor_SMD:C_1206_3216Metric_Pad1.33x1.80mm_HandSolder -> PCM_Capacitor_SMD_AKL:C_1206_3216Metric_Pad1.42x1.75mm_HandSolder
- C2: renamed from C3; footprint Capacitor_SMD:C_1206_3216Metric_Pad1.33x1.80mm_HandSolder -> PCM_Capacitor_SMD_AKL:C_1206_3216Metric_Pad1.42x1.75mm_HandSolder
- C3: renamed from C2; footprint Capacitor_SMD:C_1206_3216Metric_Pad1.33x1.80mm_HandSolder -> PCM_Capacitor_SMD_AKL:C_1206_3216Metric_Pad1.42x1.75mm_HandSolder
- J4: renamed from J5; value Screw_Terminal_01x04 -> Panel power 1
- J5: renamed from J6; value Screw_Terminal_01x04 -> Panel power 2
- moved C1 30.6 mm to (57.0, 67.0), turned to 90 degrees
- moved C3 30.2 mm to (53.5, 67.0), turned to -90 degrees
- moved R3 4.76 mm to (61.5, 59.5), turned to 90 degrees
- moved LED1 4.75 mm to (55.2, 58.2)
- moved C10 1.75 mm to (139.2, 128.6)
- moved C11 1.75 mm to (60.8, 128.5)
- moved J3 1.03 mm to (56.5, 81.3)
- moved C4 0.50 mm to (142.4, 73.0)
- moved C5 0.50 mm to (142.4, 62.0)
- renumbered J9 to J10, J10 to J11, J1 to J2, J2 to J3, J3 to J6, J4 to J7, J7 to J8, J8 to J9, R1 to R3, R2 to R4, R3 to R5
Connections:
- net +3.3V renamed +3.3V_1
- net Net-(U1-3V3_1) renamed +3.3V_2
Routing:
- net +3.3V_2: track 29.7 -> 71.0 mm, vias 0 -> 1
- net Net-(J2-Pin_1): track 0.00 -> 33.0 mm, vias 0 -> 9
- net LED2: track 18.3 -> 40.3 mm
- net SCL: track 82.0 -> 103.3 mm
- net SDA: track 81.5 -> 101.6 mm
- net LED1: track 15.3 -> 25.8 mm
- net +3.3V_1: track 75.4 -> 85.4 mm
- net Net-(LED1-AK): track 0.00 -> 7.39 mm
- net GND: track 15.4 -> 22.6 mm, vias 7 -> 9
- net +5V: track 278.2 -> 284.4 mm
- net BUF_P0_CLOCK: track 19.8 -> 19.2 mm
- added copper zone on B.Cu, net Net-(J2-Pin_1)
Other:
- board text added: "+3.3V"
- board text added: "HUB75(E) Controller V1.0 ©2025 Marc Schöndorf"
- board text added: "INPUT POWER"
- board text added: "STATUS"

Commit message: Added serial number to board
Parts:
- moved G*** 1.00 mm to (88.5, 66.0)
- moved G*** 1.00 mm to (112.0, 65.5)
- moved G*** 1.00 mm to (99.5, 65.0)

Commit message: Added plots and BOM
Parts:
- moved U3 45.5 mm to (154.9, 90.2)
- moved C1 45.5 mm to (102.5, 67.0)
- moved C10 45.5 mm to (184.8, 128.6)
- moved C11 45.5 mm to (106.2, 128.5)
- moved C2 45.5 mm to (166.2, 84.5)
- moved C3 45.5 mm to (99.0, 67.0)
- moved C4 45.5 mm to (187.9, 73.0)
- moved C5 45.5 mm to (187.9, 62.0)
- moved C6 45.5 mm to (127.2, 91.0)
- moved C7 45.5 mm to (127.2, 97.0)
- moved C8 45.5 mm to (160.0, 97.0)
- moved C9 45.5 mm to (188.0, 86.8)
- moved F1 45.5 mm to (126.5, 138.2)
- moved G*** 45.5 mm to (145.5, 103.5)
- moved G*** 45.5 mm to (134.0, 66.0)
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